Commit message: Add Nav2 navigation, my_world map and base_footprint frame

File: urdf/mobile_robot_urdf.xacro (robot description, xacro)
@@ -515,3 +515,9 @@
   <limit effort="1.0" velocity="3.3"/>
 </joint>
+<link name="base_footprint"/>
+<joint name="base_footprint_joint" type="fixed">
+  <parent link="base_footprint"/>
+  <child link="base_link"/>
+  <origin xyz="0.03 0 0.068" rpy="0 0 0"/>
+</joint>
 </robot>
